Commit message: Fixed kobuki base drifting by adding a 'mu' value of 100000 in each wheel link and fixed the gazebo reference name by adding '/{robot_name}' in file 'locobot_kobuki.urdf.xacro'.
Fixed point cloud position given by a typo in file 'pan_and_tilt.urdf'.

File: interbotix_ros_xslocobots/interbotix_xslocobot_descriptions/urdf/kobuki_version/locobot_kobuki.urdf.xacro (robot description, xacro)
@@ -149,7 +149,8 @@
     </inertial>
   </link>
-  <gazebo reference="wheel_left_link">
-    <mu1>1.0</mu1>
-    <mu2>1.0</mu2>
+  <gazebo reference="${robot_name}/wheel_left_link">
+    <!-- This friction pamareter don't contain reliable data!! -->
+    <mu1>100000.0</mu1>
+    <mu2>100000.0</mu2>
     <kp>1000000.0</kp>
     <kd>100.0</kd>
@@ -212,5 +213,47 @@
     </inertial>
   </link>
-  <gazebo reference="wheel_right_link">
+  <gazebo reference="${robot_name}/wheel_right_link">
+    <!-- This friction pamareter don't contain reliable data!! -->
+    <mu1>100000.0</mu1>
+    <mu2>100000.0</mu2>
+    <kp>1000000.0</kp>
+    <kd>100.0</kd>
+    <minDepth>0.001</minDepth>
+    <maxVel>1.0</maxVel>
+  </gazebo>
+  <joint name="caster_front_joint" type="fixed">
+    <origin
+      rpy="-1.57079632679 0 0"
+      xyz="0.115 0.0 0.007"/>
+    <parent
+      link="${robot_name}/base_link"/>
+    <child
+      link="${robot_name}/caster_front_link"/>
+  </joint>
+  <link name="${robot_name}/caster_front_link">
+    <collision>
+      <origin
+        rpy="0 0 0"
+        xyz="0 0 0"/>
+      <geometry>
+        <cylinder
+          length="0.0176"
+          radius="0.017"/>
+      </geometry>
+    </collision>
+    <inertial>
+      <origin
+        xyz="0 0 0"/>
+      <mass value="0.01"/>
+      <inertia
+        ixx="0.001"
+        ixy="0.0"
+        ixz="0.0"
+        iyy="0.001"
+        iyz="0.0"
+        izz="0.001"/>
+    </inertial>
+  </link>
+  <gazebo reference="${robot_name}/caster_front_link">
     <mu1>1.0</mu1>
     <mu2>1.0</mu2>
@@ -220,14 +263,14 @@
     <maxVel>1.0</maxVel>
   </gazebo>
-  <joint name="caster_front_joint" type="fixed">
+  <joint name="caster_back_joint" type="fixed">
     <origin
       rpy="-1.57079632679 0 0"
-      xyz="0.115 0.0 0.007"/>
-    <parent
-      link="${robot_name}/base_link"/>
-    <child
-      link="${robot_name}/caster_front_link"/>
-  </joint>
-  <link name="${robot_name}/caster_front_link">
+      xyz="-0.135 0.0 0.009"/>
+    <parent
+      link="${robot_name}/base_link"/>
+    <child
+      link="${robot_name}/caster_back_link"/>
+  </joint>
+  <link name="${robot_name}/caster_back_link">
     <collision>
       <origin
@@ -253,48 +296,7 @@
     </inertial>
   </link>
-  <gazebo reference="caster_front_link">
-    <mu1>0.0</mu1>
-    <mu2>0.0</mu2>
-    <kp>1000000.0</kp>
-    <kd>100.0</kd>
-    <minDepth>0.001</minDepth>
-    <maxVel>1.0</maxVel>
-  </gazebo>
-  <joint name="caster_back_joint" type="fixed">
-    <origin
-      rpy="-1.57079632679 0 0"
-      xyz="-0.135 0.0 0.009"/>
-    <parent
-      link="${robot_name}/base_link"/>
-    <child
-      link="${robot_name}/caster_back_link"/>
-  </joint>
-  <link name="${robot_name}/caster_back_link">
-    <collision>
-      <origin
-        rpy="0 0 0"
-        xyz="0 0 0"/>
-      <geometry>
-        <cylinder
-          length="0.0176"
-          radius="0.017"/>
-      </geometry>
-    </collision>
-    <inertial>
-      <origin
-        xyz="0 0 0"/>
-      <mass value="0.01"/>
-      <inertia
-        ixx="0.001"
-        ixy="0.0"
-        ixz="0.0"
-        iyy="0.001"
-        iyz="0.0"
-        izz="0.001"/>
-    </inertial>
-  </link>
-  <gazebo reference="caster_back_link">
-    <mu1>0.0</mu1>
-    <mu2>0.0</mu2>
+  <gazebo reference="${robot_name}/caster_back_link">
+    <mu1>1.0</mu1>
+    <mu2>1.0</mu2>
     <kp>1000000.0</kp>
     <kd>100.0</kd>

File: interbotix_ros_xslocobots/interbotix_xslocobot_descriptions/urdf/pan_and_tilt.urdf.xacro (robot description, xacro)
@@ -230,5 +230,5 @@
           <depthImageCameraInfoTopicName>aligned_depth_to_color/camera_info</depthImageCameraInfoTopicName>
           <pointCloudTopicName>depth_registered/points</pointCloudTopicName>
-          <frameName>${robot_name}/camera_depth_link</frameName>
+          <frame_name>${robot_name}/camera_depth_link</frame_name>
           <pointCloudCutoff>0.01</pointCloudCutoff>
           <pointCloudCutoffMax>10</pointCloudCutoffMax>
